Commit message: fix Link_Waist_Pitch com position value error

File: urdf/igris_c_v2.urdf (robot description, URDF)
Before this commit: robot IGRIS_C, 34 links, 33 joints
Links:
- link Left_Hand: geometry collision box size=0.15 0.05 0.2; visual mesh filename=package://igris_c_description/meshes/igris_c_v2/Hand_Left.s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 scale=0.01 0.01 0.01
- link Link_Ankle_Pitch_Left: geometry visual mesh filename=package://igris_c_description/meshes/igris_c_v2/Ankle_Pitch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 scale=0.01 0.01 0.01
- link Link_Ankle_Pitch_Right: geometry visual mesh filename=package://igris_c_description/meshes/igris_c_v2/Ankle_Pitch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 scale=0.01 0.01 0.01
- link Link_Ankle_Roll_Left: mass 0.459 -> 0.579; geometry collision box size=0.2 0.07 0.014; visual mesh filename=package://igris_c_description/meshes/igris_c_v2/Ankle_Roll_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 scale=0.01 0.01 0.01
- link Link_Ankle_Roll_Right: mass 0.459 -> 0.579; geometry collision box size=0.2 0.07 0.014; visual mesh filename=package://igris_c_description/meshes/igris_c_v2/Ankle_Roll_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 scale=0.01 0.01 0.01
- link Link_Elbow_Pitch_Left: geometry visual mesh filename=package://igris_c_description/meshes/igris_c_v2/Elbow_Pitch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 scale=0.01 0.01 0.01
- link Link_Elbow_Pitch_Right: geometry visual mesh filename=package://igris_c_description/meshes/igris_c_v2/Elbow_Pitch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 scale=0.01 0.01 0.01
- link Link_Hip_Pitch_Left: geometry visual mesh filename=package://igris_c_description/meshes/igris_c_v2/Hip_Pitch_L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 scale=0.01 0.01 0.01
- link Link_Hip_Pitch_Right: geometry visual mesh filename=package://igris_c_description/meshes/igris_c_v2/Hip_Pitch_R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 scale=0.01 0.01 0.01
- link Link_Hip_Roll_Left: geometry collision box size=0.16 0.12 0.12; visual mesh filename=package://igris_c_description/meshes/igris_c_v2/Hip_Roll_Le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 scale=0.01 0.01 0.01
- link Link_Hip_Roll_Right: geometry collision box size=0.16 0.12 0.12; visual mesh filename=package://igris_c_description/meshes/igris_c_v2/Hip_Roll_Ri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 scale=0.01 0.01 0.01
- link Link_Hip_Yaw_Left: geometry visual mesh filename=package://igris_c_description/meshes/igris_c_v2/Hip_Yaw_Lef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 scale=0.01 0.01 0.01
- link Link_Hip_Yaw_Right: geometry visual mesh filename=package://igris_c_description/meshes/igris_c_v2/Hip_Yaw_Rig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 scale=0.01 0.01 0.01
- link Link_Knee_Pitch_Left: geometry collision box size=0.15 0.1 0.25; visual mesh filename=package://igris_c_description/meshes/igris_c_v2/Knee_Pitch_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 scale=0.01 0.01 0.01
- link Link_Knee_Pitch_Right: geometry collision box size=0.15 0.1 0.25; visual mesh filename=package://igris_c_description/meshes/igris_c_v2/Knee_Pitch_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 scale=0.01 0.01 0.01
- link Link_Neck_Pitch: geometry collision box size=0.2 0.15 0.18; visual mesh filename=package://igris_c_description/meshes/igris_c_v2/Neck_Pitch.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 scale=0.01 0.01 0.01
- link Link_Neck_Yaw: geometry visual mesh filename=package://igris_c_description/meshes/igris_c_v2/Neck_Yaw.stl scale=0.01 0.01 0.01
- link Link_Shoulder_Pitch_Left: geometry visual mesh filename=package://igris_c_description/meshes/igris_c_v2/Shoulder_Pi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 scale=0.01 0.01 0.01
- link Link_Shoulder_Pitch_Right: geometry visual mesh filename=package://igris_c_description/meshes/igris_c_v2/Shoulder_Pi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 scale=0.01 0.01 0.01
- link Link_Shoulder_Roll_Left: geometry visual mesh filename=package://igris_c_description/meshes/igris_c_v2/Shoulder_Ro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 scale=0.01 0.01 0.01
- link Link_Shoulder_Roll_Right: geometry visual mesh filename=package://igris_c_description/meshes/igris_c_v2/Shoulder_Ro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 scale=0.01 0.01 0.01
- link Link_Shoulder_Yaw_Left: geometry visual mesh filename=package://igris_c_description/meshes/igris_c_v2/Shoulder_Ya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 scale=0.01 0.01 0.01
- link Link_Shoulder_Yaw_Right: geometry visual mesh filename=package://igris_c_description/meshes/igris_c_v2/Shoulder_Ya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 scale=0.01 0.01 0.01
- link Link_Waist_Pitch: geometry visual mesh filename=package://igris_c_description/meshes/igris_c_v2/Waist_Pitch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 scale=0.01 0.01 0.01
- link Link_Waist_Roll: geometry visual mesh filename=package://igris_c_description/meshes/igris_c_v2/Waist_Roll_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 scale=0.01 0.01 0.01
- link Link_Waist_Yaw: geometry visual mesh filename=package://igris_c_description/meshes/igris_c_v2/Waist_Yaw_B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 scale=0.01 0.01 0.01
- link Link_Wrist_Pitch_Left: geometry visual mesh filename=package://igris_c_description/meshes/igris_c_v2/Wrist_Pitch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 scale=0.01 0.01 0.01
- link Link_Wrist_Pitch_Right: geometry visual mesh filename=package://igris_c_description/meshes/igris_c_v2/Wrist_Pitch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 scale=0.01 0.01 0.01
- link Link_Wrist_Roll_Left: geometry visual mesh filename=package://igris_c_description/meshes/igris_c_v2/Wrist_Roll_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 scale=0.01 0.01 0.01
- link Link_Wrist_Roll_Right: geometry visual mesh filename=package://igris_c_description/meshes/igris_c_v2/Wrist_Roll_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 scale=0.01 0.01 0.01
- link Link_Wrist_Yaw_Left: geometry collision cylinder length=0.24 radius=0.05; visual mesh filename=package://igris_c_description/meshes/igris_c_v2/Wrist_Yaw_L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 scale=0.01 0.01 0.01
- link Link_Wrist_Yaw_Right: geometry collision cylinder length=0.24 radius=0.05; visual mesh filename=package://igris_c_description/meshes/igris_c_v2/Wrist_Yaw_R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 scale=0.01 0.01 0.01
- link Right_Hand: geometry collision box size=0.15 0.05 0.2; visual mesh filename=package://igris_c_description/meshes/igris_c_v2/Hand_Right.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 scale=0.01 0.01 0.01
- link base_link: geometry collision box size=0.22 0.23 0.33; visual mesh filename=package://igris_c_description/meshes/igris_c_v2/Waist_Yaw.s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 scale=0.01 0.01 0.01

File: urdf/igris_c_v2_parallel.urdf (robot description, URDF)
Before this commit: robot igris_c_v2_parallel, 70 links, 69 joints
Links:
- link Left_Hand: geometry collision mesh filename=package://igris_c_description/meshes/igris_c_v2/Hand_Left.s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 scale=0.01 0.01 0.01; visual mesh filename=package://igris_c_description/meshes/igris_c_v2/Hand_Left.s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 scale=0.01 0.01 0.01
- link Link_Ankle_Flange_In_Left: geometry collision mesh filename=package://igris_c_description/meshes/igris_c_v2/Ankle_Flang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 scale=0.01 0.01 0.01; visual mesh filename=package://igris_c_description/meshes/igris_c_v2/Ankle_Flang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 scale=0.01 0.01 0.01
- link Link_Ankle_Flange_In_Right: geometry collision mesh filename=package://igris_c_description/meshes/igris_c_v2/Ankle_Flang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 scale=0.01 0.01 0.01; visual mesh filename=package://igris_c_description/meshes/igris_c_v2/Ankle_Flang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 scale=0.01 0.01 0.01
- link Link_Ankle_Flange_Out_Left: geometry collision mesh filename=package://igris_c_description/meshes/igris_c_v2/Ankle_Flang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 scale=0.01 0.01 0.01; visual mesh filename=package://igris_c_description/meshes/igris_c_v2/Ankle_Flang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 scale=0.01 0.01 0.01
- link Link_Ankle_Flange_Out_Right: geometry collision mesh filename=package://igris_c_description/meshes/igris_c_v2/Ankle_Flang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 scale=0.01 0.01 0.01; visual mesh filename=package://igris_c_description/meshes/igris_c_v2/Ankle_Flang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 scale=0.01 0.01 0.01
- link Link_Ankle_Parallel_In_Left: geometry collision mesh filename=package://igris_c_description/meshes/igris_c_v2/Ankle_Paral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 scale=0.01 0.01 0.01; visual mesh filename=package://igris_c_description/meshes/igris_c_v2/Ankle_Paral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 scale=0.01 0.01 0.01
- link Link_Ankle_Parallel_In_Right: geometry collision mesh filename=package://igris_c_description/meshes/igris_c_v2/Ankle_Paral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 scale=0.01 0.01 0.01; visual mesh filename=package://igris_c_description/meshes/igris_c_v2/Ankle_Paral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 scale=0.01 0.01 0.01
- link Link_Ankle_Parallel_Out_Left: geometry collision mesh filename=package://igris_c_description/meshes/igris_c_v2/Ankle_Paral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 scale=0.01 0.01 0.01; visual mesh filename=package://igris_c_description/meshes/igris_c_v2/Ankle_Paral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 scale=0.01 0.01 0.01
- link Link_Ankle_Parallel_Out_Right: geometry collision mesh filename=package://igris_c_description/meshes/igris_c_v2/Ankle_Paral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 scale=0.01 0.01 0.01; visual mesh filename=package://igris_c_description/meshes/igris_c_v2/Ankle_Paral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 scale=0.01 0.01 0.01
- link Link_Ankle_Pitch_Left: geometry collision mesh filename=package://igris_c_description/meshes/igris_c_v2/Ankle_Pitch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 scale=0.01 0.01 0.01; visual mesh filename=package://igris_c_description/meshes/igris_c_v2/Ankle_Pitch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 scale=0.01 0.01 0.01
- link Link_Ankle_Pitch_Right: geometry collision mesh filename=package://igris_c_description/meshes/igris_c_v2/Ankle_Pitch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 scale=0.01 0.01 0.01; visual mesh filename=package://igris_c_description/meshes/igris_c_v2/Ankle_Pitch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 scale=0.01 0.01 0.01
- link Link_Ankle_Roll_Left: geometry collision mesh filename=package://igris_c_description/meshes/igris_c_v2/Ankle_Roll_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 scale=0.01 0.01 0.01; visual mesh filename=package://igris_c_description/meshes/igris_c_v2/Ankle_Roll_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 scale=0.01 0.01 0.01
- link Link_Ankle_Roll_Right: geometry collision mesh filename=package://igris_c_description/meshes/igris_c_v2/Ankle_Roll_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 scale=0.01 0.01 0.01; visual mesh filename=package://igris_c_description/meshes/igris_c_v2/Ankle_Roll_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 scale=0.01 0.01 0.01
- link Link_Elbow_Pitch_Left: geometry collision mesh filename=package://igris_c_description/meshes/igris_c_v2/Elbow_Pitch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 scale=0.01 0.01 0.01; visual mesh filename=package://igris_c_description/meshes/igris_c_v2/Elbow_Pitch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 scale=0.01 0.01 0.01
- link Link_Elbow_Pitch_Right: geometry collision mesh filename=package://igris_c_description/meshes/igris_c_v2/Elbow_Pitch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 scale=0.01 0.01 0.01; visual mesh filename=package://igris_c_description/meshes/igris_c_v2/Elbow_Pitch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 scale=0.01 0.01 0.01
- link Link_Hip_Pitch_Left: geometry collision mesh filename=package://igris_c_description/meshes/igris_c_v2/Hip_Pitch_L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 scale=0.01 0.01 0.01; visual mesh filename=package://igris_c_description/meshes/igris_c_v2/Hip_Pitch_L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 scale=0.01 0.01 0.01
- link Link_Hip_Pitch_Right: geometry collision mesh filename=package://igris_c_description/meshes/igris_c_v2/Hip_Pitch_R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 scale=0.01 0.01 0.01; visual mesh filename=package://igris_c_description/meshes/igris_c_v2/Hip_Pitch_R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 scale=0.01 0.01 0.01
- link Link_Hip_Roll_Left: geometry collision mesh filename=package://igris_c_description/meshes/igris_c_v2/Hip_Roll_Le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 scale=0.01 0.01 0.01; visual mesh filename=package://igris_c_description/meshes/igris_c_v2/Hip_Roll_Le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 scale=0.01 0.01 0.01
- link Link_Hip_Roll_Right: geometry collision mesh filename=package://igris_c_description/meshes/igris_c_v2/Hip_Roll_Ri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 scale=0.01 0.01 0.01; visual mesh filename=package://igris_c_description/meshes/igris_c_v2/Hip_Roll_Ri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 scale=0.01 0.01 0.01
- link Link_Hip_Yaw_Left: geometry collision mesh filename=package://igris_c_description/meshes/igris_c_v2/Hip_Yaw_Lef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 scale=0.01 0.01 0.01; visual mesh filename=package://igris_c_description/meshes/igris_c_v2/Hip_Yaw_Lef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 scale=0.01 0.01 0.01
- link Link_Hip_Yaw_Right: geometry collision mesh filename=package://igris_c_description/meshes/igris_c_v2/Hip_Yaw_Rig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 scale=0.01 0.01 0.01; visual mesh filename=package://igris_c_description/meshes/igris_c_v2/Hip_Yaw_Rig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 scale=0.01 0.01 0.01
- link Link_Knee_Pitch_Left: geometry collision mesh filename=package://igris_c_description/meshes/igris_c_v2/Knee_Pitch_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 scale=0.01 0.01 0.01; visual mesh filename=package://igris_c_description/meshes/igris_c_v2/Knee_Pitch_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 scale=0.01 0.01 0.01
- link Link_Knee_Pitch_Right: geometry collision mesh filename=package://igris_c_description/meshes/igris_c_v2/Knee_Pitch_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 scale=0.01 0.01 0.01; visual mesh filename=package://igris_c_description/meshes/igris_c_v2/Knee_Pitch_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 scale=0.01 0.01 0.01
- link Link_Neck_Pitch: geometry collision mesh filename=package://igris_c_description/meshes/igris_c_v2/Neck_Pitch.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 scale=0.01 0.01 0.01; visual mesh filename=package://igris_c_description/meshes/igris_c_v2/Neck_Pitch.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 scale=0.01 0.01 0.01
- link Link_Neck_Yaw: geometry collision mesh filename=package://igris_c_description/meshes/igris_c_v2/Neck_Yaw.stl scale=0.01 0.01 0.01; visual mesh filename=package://igris_c_description/meshes/igris_c_v2/Neck_Yaw.stl scale=0.01 0.01 0.01
- link Link_Shoulder_Pitch_Left: geometry collision mesh filename=package://igris_c_description/meshes/igris_c_v2/Shoulder_Pi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 scale=0.01 0.01 0.01; visual mesh filename=package://igris_c_description/meshes/igris_c_v2/Shoulder_Pi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 scale=0.01 0.01 0.01
- link Link_Shoulder_Pitch_Right: geometry collision mesh filename=package://igris_c_description/meshes/igris_c_v2/Shoulder_Pi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 scale=0.01 0.01 0.01; visual mesh filename=package://igris_c_description/meshes/igris_c_v2/Shoulder_Pi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 scale=0.01 0.01 0.01
- link Link_Shoulder_Roll_Left: geometry collision mesh filename=package://igris_c_description/meshes/igris_c_v2/Shoulder_Ro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 scale=0.01 0.01 0.01; visual mesh filename=package://igris_c_description/meshes/igris_c_v2/Shoulder_Ro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 scale=0.01 0.01 0.01
- link Link_Shoulder_Roll_Right: geometry collision mesh filename=package://igris_c_description/meshes/igris_c_v2/Shoulder_Ro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 scale=0.01 0.01 0.01; visual mesh filename=package://igris_c_description/meshes/igris_c_v2/Shoulder_Ro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 scale=0.01 0.01 0.01
- link Link_Shoulder_Yaw_Left: geometry collision mesh filename=package://igris_c_description/meshes/igris_c_v2/Shoulder_Ya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 scale=0.01 0.01 0.01; visual mesh filename=package://igris_c_description/meshes/igris_c_v2/Shoulder_Ya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 scale=0.01 0.01 0.01
- link Link_Shoulder_Yaw_Right: geometry collision mesh filename=package://igris_c_description/meshes/igris_c_v2/Shoulder_Ya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 scale=0.01 0.01 0.01; visual mesh filename=package://igris_c_description/meshes/igris_c_v2/Shoulder_Ya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 scale=0.01 0.01 0.01
- link Link_Waist_Flange_Left: geometry collision mesh filename=package://igris_c_description/meshes/igris_c_v2/Waist_Flang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 scale=0.01 0.01 0.01; visual mesh filename=package://igris_c_description/meshes/igris_c_v2/Waist_Flang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 scale=0.01 0.01 0.01
- link Link_Waist_Flange_Right: geometry collision mesh filename=package://igris_c_description/meshes/igris_c_v2/Waist_Flang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 scale=0.01 0.01 0.01; visual mesh filename=package://igris_c_description/meshes/igris_c_v2/Waist_Flang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 scale=0.01 0.01 0.01
- link Link_Waist_Parallel_Left: geometry collision mesh filename=package://igris_c_description/meshes/igris_c_v2/Waist_Paral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 scale=0.01 0.01 0.01; visual mesh filename=package://igris_c_description/meshes/igris_c_v2/Waist_Paral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 scale=0.01 0.01 0.01
- link Link_Waist_Parallel_Right: geometry collision mesh filename=package://igris_c_description/meshes/igris_c_v2/Waist_Paral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 scale=0.01 0.01 0.01; visual mesh filename=package://igris_c_description/meshes/igris_c_v2/Waist_Paral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 scale=0.01 0.01 0.01
- link Link_Waist_Pitch: geometry collision mesh filename=package://igris_c_description/meshes/igris_c_v2/Waist_Pitch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 scale=0.01 0.01 0.01; visual mesh filename=package://igris_c_description/meshes/igris_c_v2/Waist_Pitch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 scale=0.01 0.01 0.01
- link Link_Waist_Roll: geometry collision mesh filename=package://igris_c_description/meshes/igris_c_v2/Waist_Roll_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 scale=0.01 0.01 0.01; visual mesh filename=package://igris_c_description/meshes/igris_c_v2/Waist_Roll_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 scale=0.01 0.01 0.01
- link Link_Waist_Yaw: geometry collision mesh filename=package://igris_c_description/meshes/igris_c_v2/Waist_Yaw_B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 scale=0.01 0.01 0.01; visual mesh filename=package://igris_c_description/meshes/igris_c_v2/Waist_Yaw_B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 scale=0.01 0.01 0.01
- link Link_Wrist_Flange_Back_Left: geometry collision mesh filename=package://igris_c_description/meshes/igris_c_v2/Wrist_Flang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 scale=0.01 0.01 0.01; visual mesh filename=package://igris_c_description/meshes/igris_c_v2/Wrist_Flang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 scale=0.01 0.01 0.01
- link Link_Wrist_Flange_Back_Right: geometry collision mesh filename=package://igris_c_description/meshes/igris_c_v2/Wrist_Flang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 scale=0.01 0.01 0.01; visual mesh filename=package://igris_c_description/meshes/igris_c_v2/Wrist_Flang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 scale=0.01 0.01 0.01
- link Link_Wrist_Flange_Front_Left: geometry collision mesh filename=package://igris_c_description/meshes/igris_c_v2/Wrist_Flang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 scale=0.01 0.01 0.01; visual mesh filename=package://igris_c_description/meshes/igris_c_v2/Wrist_Flang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 scale=0.01 0.01 0.01
- link Link_Wrist_Flange_Front_Right: geometry collision mesh filename=package://igris_c_description/meshes/igris_c_v2/Wrist_Flang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 scale=0.01 0.01 0.01; visual mesh filename=package://igris_c_description/meshes/igris_c_v2/Wrist_Flang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 scale=0.01 0.01 0.01
- link Link_Wrist_Parallel_Back_Left: geometry collision mesh filename=package://igris_c_description/meshes/igris_c_v2/Wrist_Paral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 scale=0.01 0.01 0.01; visual mesh filename=package://igris_c_description/meshes/igris_c_v2/Wrist_Paral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 scale=0.01 0.01 0.01
- link Link_Wrist_Parallel_Back_Right: geometry collision mesh filename=package://igris_c_description/meshes/igris_c_v2/Wrist_Paral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 scale=0.01 0.01 0.01; visual mesh filename=package://igris_c_description/meshes/igris_c_v2/Wrist_Paral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 scale=0.01 0.01 0.01
- link Link_Wrist_Parallel_Front_Left: geometry collision mesh filename=package://igris_c_description/meshes/igris_c_v2/Wrist_Paral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 scale=0.01 0.01 0.01; visual mesh filename=package://igris_c_description/meshes/igris_c_v2/Wrist_Paral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 scale=0.01 0.01 0.01
- link Link_Wrist_Parallel_Front_Right: geometry collision mesh filename=package://igris_c_description/meshes/igris_c_v2/Wrist_Paral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 scale=0.01 0.01 0.01; visual mesh filename=package://igris_c_description/meshes/igris_c_v2/Wrist_Paral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 scale=0.01 0.01 0.01
- link Link_Wrist_Pitch_Left: geometry collision mesh filename=package://igris_c_description/meshes/igris_c_v2/Wrist_Pitch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 scale=0.01 0.01 0.01; visual mesh filename=package://igris_c_description/meshes/igris_c_v2/Wrist_Pitch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 scale=0.01 0.01 0.01
- link Link_Wrist_Pitch_Right: geometry collision mesh filename=package://igris_c_description/meshes/igris_c_v2/Wrist_Pitch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 scale=0.01 0.01 0.01; visual mesh filename=package://igris_c_description/meshes/igris_c_v2/Wrist_Pitch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 scale=0.01 0.01 0.01
- link Link_Wrist_Roll_Left: geometry collision mesh filename=package://igris_c_description/meshes/igris_c_v2/Wrist_Roll_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 scale=0.01 0.01 0.01; visual mesh filename=package://igris_c_description/meshes/igris_c_v2/Wrist_Roll_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 scale=0.01 0.01 0.01
- link Link_Wrist_Roll_Right: geometry collision mesh filename=package://igris_c_description/meshes/igris_c_v2/Wrist_Roll_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 scale=0.01 0.01 0.01; visual mesh filename=package://igris_c_description/meshes/igris_c_v2/Wrist_Roll_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 scale=0.01 0.01 0.01
- link Link_Wrist_Universal_Back_Left: geometry collision mesh filename=package://igris_c_description/meshes/igris_c_v2/Wrist_Unive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 scale=0.01 0.01 0.01; visual mesh filename=package://igris_c_description/meshes/igris_c_v2/Wrist_Unive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 scale=0.01 0.01 0.01
- link Link_Wrist_Universal_Back_Right: geometry collision mesh filename=package://igris_c_description/meshes/igris_c_v2/Wrist_Unive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 scale=0.01 0.01 0.01; visual mesh filename=package://igris_c_description/meshes/igris_c_v2/Wrist_Unive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 scale=0.01 0.01 0.01
- link Link_Wrist_Universal_Front_Left: mass 0.002 -> 0.005; geometry collision mesh filename=package://igris_c_description/meshes/igris_c_v2/Wrist_Unive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 scale=0.01 0.01 0.01; visual mesh filename=package://igris_c_description/meshes/igris_c_v2/Wrist_Unive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 scale=0.01 0.01 0.01
- link Link_Wrist_Universal_Front_Right: mass 0.002 -> 0.005; geometry collision mesh filename=package://igris_c_description/meshes/igris_c_v2/Wrist_Unive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 scale=0.01 0.01 0.01; visual mesh filename=package://igris_c_description/meshes/igris_c_v2/Wrist_Unive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 scale=0.01 0.01 0.01
- link Link_Wrist_Yaw_Left: geometry collision mesh filename=package://igris_c_description/meshes/igris_c_v2/Wrist_Yaw_L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 scale=0.01 0.01 0.01; visual mesh filename=package://igris_c_description/meshes/igris_c_v2/Wrist_Yaw_L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 scale=0.01 0.01 0.01
- link Link_Wrist_Yaw_Right: geometry collision mesh filename=package://igris_c_description/meshes/igris_c_v2/Wrist_Yaw_R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 scale=0.01 0.01 0.01; visual mesh filename=package://igris_c_description/meshes/igris_c_v2/Wrist_Yaw_R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 scale=0.01 0.01 0.01
- link Right_Hand: geometry collision mesh filename=package://igris_c_description/meshes/igris_c_v2/Hand_Right.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 scale=0.01 0.01 0.01; visual mesh filename=package://igris_c_description/meshes/igris_c_v2/Hand_Right.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 scale=0.01 0.01 0.01
- link base_link: geometry collision mesh filename=package://igris_c_description/meshes/igris_c_v2/Waist_Yaw.s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 scale=0.01 0.01 0.01; visual mesh filename=package://igris_c_description/meshes/igris_c_v2/Waist_Yaw.s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 scale=0.01 0.01 0.01
